File: hardware/fabrication_pcb/Mini Project/Mini Project.kicad_sch (KiCad schematic)
At the start: 10 parts, among them SW1 SW_Push, SW2 SW_Push, SW3 SW_Push, SW4 SW_Push

Commit message: feat: very bad basic routing
Parts:
- removed U5: ~, MyFootprints:OLED_128x64_I2C, symbol MyComponents:OLED_128x64_I2C
- added C1: 47nF, Capacitor_THT:CP_Radial_D6.3mm_P2.50mm, symbol Device:C
- added U1: DM-OLED096-636, SH1106:MODULE_DM-OLED096-636, symbol DM-OLED096-636:DM-OLED096-636
- renumbered SW4 to BTN_BACK1, SW2 to BTN_DOWN1, SW3 to BTN_SELECT1, SW1 to BTN_UP1, U6 to Speaker1, U2 to amp1, U1 to esp32, U3 to mic1, U4 to nrf1
Connections:
- net at BTN_DOWN1.1: now also esp32.24 (D33)
- net GND: now reaches BTN_DOWN1.2
- net GND: now also BTN_BACK1.2, BTN_SELECT1.2, BTN_UP1.2, Speaker1.2 (GND), amp1.3 (GND), amp1.4 (GND), amp1.6 (GND), esp32.2 (GND), mic1.2 (GND), nrf1.2 (VCC), C1.2, U1.1 (GND)
- net at Speaker1.1 (IN): now also amp1.5 (OUT)
- net at BTN_BACK1.1: now also esp32.20 (D14)
- net amp_V: now reaches amp1.1 (VCC)
- net amp_V: now also esp32.16 (VIN)
- net dac_out: now reaches amp1.2 (IN)
- net dac_out: now also esp32.23 (D25)
- net adc_inp: now reaches mic1.1 (OUT)
- net adc_inp: now also esp32.26 (D35)
- net VCC: now reaches mic1.3 (VCC)
- net VCC: now also esp32.1 (3V3), nrf1.1 (GND), C1.1, U1.2 (VCC_IN)
- net at BTN_UP1.1: now also esp32.25 (D32)
- net at BTN_SELECT1.1: now also esp32.21 (D27)
- net CE: now reaches nrf1.3 (CE)
- net CE: now also esp32.5 (D4)
- net CSN: now reaches nrf1.4 (CSN)
- net CSN: now also esp32.8 (D5)
- net SCK: now reaches nrf1.5 (SCK)
- net SCK: now also esp32.9 (D18)
- net MOSI: now reaches nrf1.6 (MOSI)
- net MOSI: now also esp32.15 (D23)
- net MISO: now reaches nrf1.7 (MISO)
- net MISO: now also esp32.10 (D19)
- net SDA: now reaches esp32.11 (D21)
- net SDA: now also U1.4 (SDA)
- net SCL: now reaches esp32.14 (D22)
- net SCL: now also U1.3 (SCL)
Other:
- moved on the sheet: BTN_BACK1, BTN_DOWN1, BTN_SELECT1, BTN_UP1, Speaker1, amp1, esp32, mic1, nrf1
